File: Eagle/12VAttinyDischargeChecker-A2.brd (EAGLE design)
At the start: 100.3 x 70 mm, 26 parts

Commit message: modificati circuiti
Parts:
- added E$15, E$16, E$19, E$20, E$21, E$25: (no value), eagle-ltspice:0204/7
- added E$24, E$38, E$40, E$41: (no value), con-lstb:MA06-1
- added E$27: (no value), 74xx-us:DIL28-3
- added E$32: (no value), LSGPackages:WIRELESS-TX-FLAT
- added E$33, E$34, E$36, E$37, E$39, E$42, E$43: (no value), testpad:P1-17Y
- added E$46, E$47, E$48, E$49, E$50, E$51: (no value), con-lstb:MA03-1
- added E$61: (no value), con-3m:PAK100/2500-10
- E$1, E$10, E$11, E$12: device LSGPackages:WIRELESS-RX-FLAT -> eagle-ltspice:0204/7
- E$13: device LSGPackages:WIRELESS-TX-FLAT -> eagle-ltspice:0204/7
- E$14: device con-lsta:FE20 -> eagle-ltspice:0204/7
- E$2: device LSGPackages:WIRELESS-TX-FLAT -> 74xx-us:DIL08
- E$3, E$4, E$5, E$6, E$7: device LSGPackages:WIRELESS-TX-FLAT -> 74xx-us:DIL28-3
- E$45: device 74xx-us:DIL08 -> testpad:P1-17Y
- E$8, E$9: device LSGPackages:WIRELESS-RX-FLAT -> con-lstb:MA04-1
- moved E$9 69.1 mm to (98.1, 31.4)
- moved E$6 58.6 mm to (77.5, 61.0), turned to 180 degrees
- moved E$14 49.5 mm to (43.8, 62.9), turned to 270 degrees
- moved E$1 44.0 mm to (44.1, 34.3), turned to 270 degrees
- moved E$13 40.7 mm to (47.6, 62.9), turned to 270 degrees
- moved E$7 34.2 mm to (77.5, 47.6), turned to 180 degrees
- moved E$5 33.4 mm to (24.1, 61.0)
- moved E$12 32.8 mm to (47.6, 46.4)
- moved E$8 31.0 mm to (2.86, 31.4), turned to 90 degrees
- moved E$3 26.5 mm to (24.1, 34.9)
- moved E$4 23.9 mm to (24.1, 48.3), turned to 0 degrees
- moved E$10 20.6 mm to (47.9, 34.3)
- moved E$11 19.0 mm to (43.8, 46.4), turned to 270 degrees
- moved E$45 15.1 mm to (52.1, 5.71), turned to 0 degrees
- moved E$2 5.68 mm to (6.35, 5.71)
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Connections:
- removed net S$11: E$1.P$1, E$14.12
- removed net S$16: E$10.P$4, E$14.7
- new net S$19: E$13.2, E$14.2, E$5.13
- new net S$20: E$15.2, E$16.2, E$6.13
- new net S$21: E$19.2, E$20.2, E$7.13
- new net S$22: E$21.2, E$25.2, E$27.13
- new net S$23: E$11.1, E$13.1, E$24.6, E$4.22
- new net S$24: E$14.1, E$15.1, E$38.6, E$5.22
- new net S$25: E$16.1, E$19.1, E$40.6, E$6.22
- new net S$26: E$20.1, E$21.1, E$41.6, E$7.22
- new net S$27: E$38.4, E$5.12
- new net S$28: E$40.1, E$6.7
- new net S$30: E$40.3, E$6.11
- new net S$31: E$40.5, E$6.12
- new net S$32: E$41.1, E$7.7
- new net S$34: E$41.3, E$7.11
- new net S$35: E$41.5, E$7.12
- new net S$36: E$27.7, E$9.4
- new net S$37: E$25.1, E$27.22, E$9.1
- new net S$38: E$27.11, E$9.3
- new net S$39: E$27.12, E$9.2
- net S$10: now also E$10.1, E$37.TP; no longer E$14.13, E$9.P$1
- net S$12: now also E$24.1, E$4.7; no longer E$12.P$1, E$14.11
- net S$13: now also E$24.3, E$4.11; no longer E$10.P$1, E$14.10
- net S$14: now also E$24.4, E$4.12; no longer E$14.9, E$8.P$1
- net S$15: now also E$38.1, E$5.7; no longer E$12.P$4, E$14.8
- net S$17: now also E$38.2, E$5.11; no longer E$14.6, E$8.P$4
- net S$2: now also E$1.1, E$12.1, E$2.4, E$3.22, E$32.P$3, E$36.TP, E$8.4; no longer E$11.P$4, E$14.20
- net S$3: now also E$2.5, E$32.P$2; no longer E$14.19, E$9.P$4
- net S$4: now also E$1.2, E$10.2, E$3.13; no longer E$1.P$4, E$14.18
- net S$5: now also E$11.2, E$12.2, E$4.13; no longer E$11.P$3, E$14.17
- net S$7: now also E$3.11, E$8.2; no longer E$14.16, E$9.P$3
- net S$8: now also E$2.8, E$3.7, E$32.P$1, E$34.TP, E$8.3; no longer E$1.P$3, E$14.15
- net S$9: now also E$3.12, E$8.1; no longer E$11.P$1, E$14.14
Other:
- board text added: "-"
- board text added: "0v"
- board text added: "14v"
- board text added: "28v"
- board text added: "42v"
- board text added: "56v"
- board text added: "70v"
- board text added: "84v"
- board text added: "A"
- board text added: "B"
- board text added: "Bi"
- board text added: "G"
- board text added: "M"
- board text added: "R"
- board text added: "V"
- board text added: "Vi"

Commit message: .
Parts:
- added E$52, E$53, E$54, E$55, E$56, E$57, E$58, E$59, E$60, E$62, E$63, E$64, E$65, E$66, E$67, E$68: (no value), testpad:P1-17Y
- moved E$26 32.7 mm to (98.1, 47.6)
- moved E$28 27.4 mm to (117.6, 16.0)
- moved E$9 6.03 mm to (98.1, 37.5)
- moved E$41 5.75 mm to (103.7, 44.0)
- moved E$36 2.62 mm to (34.0, 8.26)
- moved E$37 2.62 mm to (41.6, 8.26)
- moved E$43 2.62 mm to (45.1, 8.26)
- moved E$45 2.62 mm to (52.7, 8.26)
- moved E$33 2.62 mm to (34.0, 26.0)
- moved E$34 2.62 mm to (41.6, 26.0)
- moved E$39 2.62 mm to (45.1, 26.0)
- moved E$42 2.62 mm to (52.7, 26.0)
- moved E$49 1.93 mm to (71.1, 3.49)
- moved E$51 1.93 mm to (93.0, 3.49)
- moved E$50 1.93 mm to (81.9, 3.17)
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Connections:
- net S$10: now also E$46.3
- net S$12: now also E$53.TP
- net S$2: now also E$46.1
- net S$26: now also E$26.1, E$55.TP; no longer E$41.6
- net S$32: now also E$26.4; no longer E$41.1
- net S$34: now also E$26.3; no longer E$41.3
- net S$35: now also E$26.2; no longer E$41.5
- net S$37: now also E$54.TP
Other:
- board text added: "Coordinator"
- board text added: "In+"
- board text added: "In-"
- board text added: "Out+"
