File: Eagle/12VAttinyDischargeChecker-B2.brd (EAGLE design)
At the start: 100.3 x 70 mm, 26 parts

Commit message: modificati circuiti
Parts:
- removed E$13: (no value), LSGPackages:WIRELESS-TX-FLAT
- removed E$45: (no value), 74xx-us:DIL08
- added E$15, E$16, E$19: (no value), con-lsta:FE12
- E$10, E$12, E$8: device LSGPackages:WIRELESS-RX-FLAT -> LSGPackages:WIRELESS-TX-FLAT
- E$14: device con-lsta:FE20 -> con-lsta:FE12
- E$2, E$5, E$7: device LSGPackages:WIRELESS-TX-FLAT -> LSGPackages:WIRELESS-RX-FLAT
- moved E$8 59.0 mm to (67.9, 15.9), turned to 180 degrees
- moved E$9 48.4 mm to (81.3, 50.8)
- moved E$7 38.7 mm to (85.7, 20.3)
- moved E$11 36.4 mm to (48.9, 20.3)
- moved E$6 36.1 mm to (31.1, 41.9), turned to 180 degrees
- moved E$4 35.9 mm to (29.8, 59.1), turned to 0 degrees
- moved E$5 33.1 mm to (48.9, 54.6), turned to 270 degrees
- moved E$12 25.0 mm to (66.7, 33.0), turned to 0 degrees
- moved E$10 17.3 mm to (68.6, 52.7), turned to 90 degrees
- moved E$2 15.4 mm to (16.5, 24.1)
- moved E$3 13.3 mm to (29.2, 22.2), turned to 270 degrees
- moved E$14 12.2 mm to (97.2, 53.3)
- moved E$1 6.98 mm to (12.1, 54.6)
Connections:
- new net S$18: E$11.P$1, E$12.P$1, E$16.11
- new net S$19: E$11.P$4, E$12.P$3, E$16.12
- new net S$20: E$10.P$3, E$14.12, E$9.P$4
- new net S$21: E$10.P$1, E$14.10, E$9.P$1
- new net S$22: E$10.P$2, E$14.8
- new net S$23: E$12.P$2, E$14.3
- new net S$24: E$16.9, E$8.P$2
- new net S$25: E$16.6, E$7.P$3
- new net S$26: E$15.12, E$5.P$3
- new net S$27: E$11.P$3, E$14.1
- net S$10: now also E$15.3, E$2.P$1, E$3.P$1; no longer E$14.13, E$9.P$1
- net S$11: now also E$15.2, E$2.P$3; no longer E$1.P$1, E$14.12
- net S$12: now also E$1.P$3, E$19.11; no longer E$12.P$1, E$14.11
- net S$13: now also E$16.7, E$7.P$1, E$8.P$1; no longer E$10.P$1, E$14.10
- net S$14: now also E$15.7, E$3.P$2; no longer E$14.9, E$8.P$1
- net S$15: now also E$19.9, E$4.P$2; no longer E$12.P$4, E$14.8
- net S$16: now also E$19.5, E$6.P$2; no longer E$10.P$4, E$14.7
- net S$17: now also E$14.11, E$9.P$3; no longer E$14.6, E$8.P$4
- net S$2: now also E$1.P$4, E$19.12, E$4.P$3; no longer E$11.P$4, E$14.20
- net S$3: now also E$19.6, E$5.P$1, E$6.P$1; no longer E$14.19, E$9.P$4
- net S$4: now also E$19.8; no longer E$1.P$4, E$14.18
- net S$5: now also E$16.5, E$7.P$4, E$8.P$3; no longer E$11.P$3, E$14.17
- net S$7: now also E$1.P$1, E$19.10, E$4.P$1; no longer E$14.16, E$9.P$3
- net S$8: now also E$19.7, E$5.P$4, E$6.P$3; no longer E$1.P$3, E$14.15
- net S$9: now also E$15.1, E$2.P$4, E$3.P$3; no longer E$11.P$1, E$14.14
Routing:
- net S$23: track 0.00 -> 75.3 mm
- net S$16: track 0.00 -> 63.9 mm
- net S$8: track 0.00 -> 60.8 mm
- net S$18: track 0.00 -> 51.5 mm
- net S$27: track 0.00 -> 50.6 mm
- net S$3: track 0.00 -> 47.7 mm
- net S$19: track 0.00 -> 46.7 mm
- net S$26: track 0.00 -> 45.7 mm
- net S$5: track 0.00 -> 39.9 mm
- net S$2: track 0.00 -> 37.6 mm
- net S$7: track 0.00 -> 37.0 mm
- net S$13: track 0.00 -> 33.9 mm
- net S$9: track 0.00 -> 33.1 mm
- net S$20: track 0.00 -> 32.9 mm
- net S$10: track 0.00 -> 30.6 mm
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Other:
- board text added: "B0"
- board text added: "B1"
- board text added: "B2"
- board text added: "B3"
- board text added: "B4"
- board text added: "B5"

Commit message: .
Parts:
- removed E$15: (no value), con-lsta:FE12
- removed E$17: (no value), eagle-ltspice:0204/7
- removed E$18: (no value), transistor-fet:TO92-
- removed E$22: (no value), pinhead:1X01/90
- removed E$23: (no value), ref-packages-longpad:E5-8,5
- removed E$28: (no value), con-lstb:MA06-1
- removed E$29: (no value), con-wago-508:W237-132
- removed E$30: (no value), discrete:RS-2,5
- removed E$31: (no value), pinhead:2X02/90
- removed E$35: (no value), con-lstb:MA04-1
- removed E$44: (no value), testpad:P1-17Y
- added E$13, E$20: (no value), con-lstb:MA04-1
- E$14, E$16, E$19: device con-lsta:FE12 -> con-lstb:MA04-1
- moved E$16 103.9 mm to (3.81, 62.2)
- moved E$26 47.4 mm to (96.5, 62.2)
- moved E$19 16.6 mm to (3.81, 36.8)
- moved E$14 16.5 mm to (96.5, 36.8)
Connections:
- removed net S$4: E$19.8
- net S$10: now also E$19.3; no longer E$15.3
- net S$11: now also E$19.2; no longer E$15.2
- net S$12: now also E$16.3; no longer E$19.11
- net S$13: now also E$14.3; no longer E$16.7
- net S$14: now also E$19.4; no longer E$15.7
- net S$15: now also E$16.1; no longer E$19.9
- net S$16: now also E$20.2; no longer E$19.5
- net S$17: now also E$26.3; no longer E$14.11
- net S$18: now also E$13.2; no longer E$16.11
- net S$19: now also E$13.1; no longer E$16.12
- net S$2: now also E$16.4; no longer E$19.12
- net S$20: now also E$26.4; no longer E$14.12
- net S$21: now also E$26.2; no longer E$14.10
- net S$22: now also E$26.1; no longer E$14.8
- net S$23: now also E$13.3; no longer E$14.3
- net S$24: now also E$14.4; no longer E$16.9
- net S$25: now also E$14.2; no longer E$16.6
- net S$26: now also E$20.1; no longer E$15.12
- net S$27: now also E$13.4; no longer E$14.1
- net S$3: now also E$20.3; no longer E$19.6
- net S$5: now also E$14.1; no longer E$16.5
- net S$7: now also E$16.2; no longer E$19.10
- net S$8: now also E$20.4; no longer E$19.7
- net S$9: now also E$19.1; no longer E$15.1
Routing:
- net S$5: track 39.9 -> 55.4 mm
- net S$13: track 33.9 -> 47.1 mm
- net S$25: track 20.7 -> 33.0 mm
- net S$23: track 75.3 -> 86.6 mm
- net S$18: track 51.5 -> 61.2 mm
- net S$11: track 13.4 -> 22.8 mm
- net S$20: track 32.9 -> 25.8 mm
- net S$24: track 27.9 -> 34.9 mm
- net S$27: track 50.6 -> 57.5 mm
- net S$9: track 33.1 -> 39.4 mm
- net S$7: track 37.0 -> 31.5 mm
- net S$10: track 30.6 -> 35.1 mm
- net S$19: track 46.7 -> 50.8 mm
- net S$15: track 30.2 -> 26.1 mm
- net S$26: track 45.7 -> 41.9 mm
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