File: Eagle/12VAttinyDischargeChecker-SingleModule-Trasmitter12V.brd (EAGLE design)
At the start: 121.6 x 70.4 mm, 67 parts

Commit message: .
Connections:
- new net S$38: E$35.17, E$40.P$3
Routing:
- net S$38: track 0.00 -> 60.0 mm, vias 0 -> 1
- net S$32: track 0.00 -> 56.4 mm
- net S$26: track 49.3 -> 44.1 mm
- net S$20: track 87.3 -> 89.7 mm
- net S$34: track 18.3 -> 19.8 mm
- net S$21: track 51.2 -> 52.0 mm
- net S$23: track 149.4 -> 148.6 mm
- net S$28: track 3.78 -> 3.20 mm
