File: Eagle/12VAttinyDischargeChecker-SingleModuleForPcb.brd (EAGLE design)
At the start: 121.6 x 70.4 mm, 67 parts

Commit message: .
Parts:
- removed E$1, E$8: 220, eagle-ltspice:0204/7
- removed E$10, E$11, E$12, E$13: (no value), wirepad:2,54/0,8
- removed E$14: Zener 5v, ref-packages:DO35Z7
- removed E$15, E$16, E$17, E$18, E$19, E$20, E$21, E$22, E$23, E$24, E$28, E$29, E$30, E$31, E$32, E$33: (no value), wirepad:1,6/0,8
- removed E$2: (no value), 74xx-us:DIL28-3
- removed E$25, E$26: (no value), diode:DO34-5
- removed E$27, E$4, E$5, E$9: (no value), con-lsta2:FE01-1
- removed E$3: (no value), LSGPackages:WIRELESS-TX-FLAT
- removed E$48: (no value), con-3m:PAK100/2500-8
- removed E$6: Zener 12v, ref-packages:DO35Z7
- removed E$7: (no value), LSGPackages:WIRELESS-RX-FLAT
- removed E$70: (no value), atmel:LOGO
- removed E$77, E$78: (no value), pinhead:2X02/90
- E$61: value (none) -> 104
- moved E$41 46.2 mm to (60.2, 21.1)
- moved E$43 46.2 mm to (34.9, 20.8)
- moved E$44 46.2 mm to (42.5, 20.8)
- moved E$47 46.2 mm to (49.5, 20.8)
- moved E$60 46.2 mm to (27.5, 22.0)
- moved E$71 46.2 mm to (68.8, 20.8)
- moved E$82 46.2 mm to (77.1, 20.8)
- moved E$104 46.2 mm to (2.12, 13.4)
- moved E$34 46.2 mm to (62.8, 4.97)
- moved E$36 46.2 mm to (90.1, 12.3)
- moved E$39 46.2 mm to (51.4, 4.97)
- moved E$40 46.2 mm to (17.1, 15.1)
- moved E$45 46.2 mm to (34.9, 4.33)
- moved E$46 46.2 mm to (42.5, 4.33)
- moved E$49 46.2 mm to (69.2, 6.87)
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Connections:
- removed net S$10: E$19.1, E$2.14
- removed net S$11: E$18.1, E$2.13
- removed net S$12: E$17.1, E$2.12
- removed net S$13: E$16.1, E$2.11
- removed net S$14: E$2.10
- removed net S$15: E$25.C, E$26.A
- removed net S$16: E$2.3, E$27.1
- removed net S$17: E$15.1, E$2.6
- removed net S$18: E$2.1, E$29.1
- removed net S$19: E$2.19, E$31.1
- removed net S$2: E$11.1, E$2.20, E$2.7, E$3.P$1, E$7.P$1, E$8.2
- removed net S$3: E$13.1, E$4.1, E$5.1, E$6.C
- removed net S$34: E$104.ID, E$61.1
- removed net S$4: E$1.2, E$14.C, E$2.23, E$6.A
- removed net S$43: E$48.10, E$77.4
- removed net S$44: E$48.9, E$77.3
- removed net S$5: E$1.1, E$12.1, E$14.A, E$2.22, E$2.8, E$20.1, E$21.1, E$22.1, E$23.1, E$24.1, E$26.C, E$28.1, E$3.P$3, E$33.1, E$7.P$4
- removed net S$51: E$48.8, E$77.2
- removed net S$52: E$48.7, E$77.1
- removed net S$53: E$48.6, E$78.4
- removed net S$54: E$48.5, E$78.3
- removed net S$55: E$48.4, E$78.2
- removed net S$56: E$78.1
- removed net S$7: E$2.18, E$3.P$2, E$32.1
- removed net S$8: E$2.21, E$25.A, E$8.1
- removed net S$9: E$2.17, E$30.1, E$7.P$3
- new net S$1: E$104.VBUS, E$61.1
- new net S$38: E$35.17, E$40.P$3
Routing:
- net S$5: track 216.0 -> 0.00 mm
- net S$2: track 139.8 -> 0.00 mm
- net S$9: track 87.8 -> 0.00 mm
- net S$7: track 66.7 -> 0.00 mm
- net S$38: track 0.00 -> 60.0 mm, vias 0 -> 1
- net S$18: track 58.9 -> 0.00 mm
- net S$32: track 0.00 -> 56.4 mm
- net S$3: track 52.7 -> 0.00 mm
- net S$19: track 49.7 -> 0.00 mm
- net S$16: track 46.7 -> 0.00 mm
- net S$4: track 37.9 -> 0.00 mm
- net S$43: track 19.9 -> 0.00 mm
- net S$34: track 18.3 -> 0.00 mm
- net S$1: track 0.00 -> 14.8 mm
- net S$17: track 11.4 -> 0.00 mm
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Other:
- board size 121.6 x 70.4 mm -> 100.3 x 24 mm
- board text removed: "A"
- board text removed: "B"
- board text removed: "Bi"
- board text removed: "G"
- board text removed: "M"
- board text removed: "Mosi"
- board text removed: "R"
- board text removed: "V"
- board text removed: "Vi"
- board text removed: "mi"
- board text removed: "mo"
- board text removed: "rs"
- board text removed: "sck"
